File: LC86G_devboard.kicad_sch (KiCad schematic)
At the start: 14 parts, among them J1 Conn_01x09_Pin, J2 U.FL-R-SMT_10_, Q1 DTC143Z, Q2 DTC143Z, Q3 AO3415, U1 LC86G

Commit message: carga final
Parts:
- removed J1: Conn_01x09_Pin, Connector_PinHeader_2.54mm:PinHeader_1x09_P2.54mm_Vertical, symbol Connector:Conn_01x09_Pin
- added D2: LED_Small, LED_SMD:LED_0603_1608Metric, symbol Device:LED_Small
- added J3: Conn_01x10_Pin, Connector_PinHeader_2.54mm:PinHeader_1x10_P2.54mm_Vertical, symbol Connector:Conn_01x10_Pin
- added JP1: SolderJumper_2_Open, SolderJumper-2_P1.3mm_Open_TrianglePad1.0x1.5mm, symbol Jumper:SolderJumper_2_Open
- added R2: 4.7k, Resistor_SMD:R_0603_1608Metric_Pad0.98x0.95mm_HandSolder, symbol Device:R_Small
- added U2: XC6206P332MR, EasyEDA:SOT-23-3_L2.9-W1.6-P1.90-LS2.8-BR, symbol EasyEDA:XC6206P332MR
Connections:
- net V_BCKP is gone; now on net LC86G.V_BCKP: C2.1, C4.1, C6.1, D1.5 (K)
- net GND: now also J3.10 (Pin_10), JP1.2 (B), U2.1 (GND)
- net GPIO.RESET: now also J3.5 (Pin_5)
- net LC86G.1PPS: now also J3.9 (Pin_9)
- net LC86G.AADET: now also J3.6 (Pin_6)
- net LC86G.RXD: now also J3.7 (Pin_7)
- net LC86G.TXD: now also J3.8 (Pin_8)
- net LC86G.V_BCKP: now also J3.4 (Pin_4)
- net ON/OFF: now also J3.3 (Pin_3)
- net VCC: now also D2.2 (A), J3.2 (Pin_2), U2.2 (Vout)
- new net: D2.1 (K), R2.1
- new net: JP1.1 (A), R2.2
- new net LDO: J3.1 (Pin_1), U2.3 (Vin)
- no-connect marks 2 -> 3
Other:
- note added: "stackup: JLC04161H-7628 Coplanar Single Ended Impedance trace to copper: 0.5080 Trace Width: 0.3424"
